File: AC-FR/ACFR-PCB/ACFR-PCB.kicad_sch (KiCad schematic)
At the start: 42 parts, among them J1 USB4105-GF-A, J2 JST-SM04B-SRSS, J3 JST-PH, Q1 DMP2045U-7, SW1 PTS636 SK25F, SW2 PTS636 SK25F, U1 ESP32-S3R8, U2 W25Q128JVPIQ, U3 BMP390, U4 MAX1704x, U5 AP2112K-3.3TRG1, U6 AP2112K-3.3TRG1, Y1 ECS-400-8-36B-7KY

Commit message: Add High G Accel, clean schematic
Parts:
- removed R8: 10k, Capacitor_SMD:C_0603_1608Metric, symbol Device:R
- added C17, C19: 100nF, Capacitor_SMD:C_0603_1608Metric, symbol Device:C
- added C18: 0.5 F, symbol Device:C_Polarized_US
- added U7: LIS3DH, Package_LGA:LGA-16_3x3mm_P0.5mm_LayoutBorder3x5y, symbol Sensor_Motion:LIS3DH
- added U8: H3LIS331DL, symbol besserLib:H3LIS331DL
Connections:
- net CTG is gone; now on net +3V3_2: C1.2, C10.2, C11.1, C13.2, C14.1, C15.1, C16.2, C2.1, C3.2, C4.2, C5.2, C6.2, C7.1, C8.2, C9.1, D1.2 (VSS), J1.A1 (GND), J1.A12 (GND), J1.B1 (GND), J1.B12 (GND), J2.1 (Pin_1), J3.2 (Pin_2), R5.2, R6.2, R7.2, SW1.2 (B), SW2.1 (A), U1.57 (GND), U2.4 (GND), U3.3 (VSS), U3.8 (VSS), U3.9 (VSS), U4.1 (CTG), U4.4 (GND), U4.6 (QSTRT), U5.2 (GND), U6.2 (GND), Y1.2, Y1.4
- net +3V3_2: now also C12.2, C17.1, C17.2, C18.2, C19.1, C19.2, U7.1 (VDD_IO), U7.10 (GND), U7.12 (GND), U7.14 (VDD), U7.5 (GND), U7.7 (SDO/SA0), U7.8 (CS), U8.1 (VDD_IO), U8.10 (NC), U8.12 (GND), U8.13 (GND), U8.14 (VDD), U8.15 (NC), U8.16 (GND), U8.5 (GND), U8.7 (SA0), U8.8 (CS)
- net SCL: now also U7.4 (SCL/SPC), U8.4 (SCL)
- net SDA: now also U7.6 (SDA/SDI/SDO), U8.6 (SDA)
- net VBAT: now also C18.1
- net VHIGH: now also U6.3 (EN)
- net XTAL_P: now also C12.1
- net 3V3_2_EN: no longer names the net of U1.43 (GPIO38)
- net 3V3_2_EN: no longer U6.3 (EN)
- net ACC_INT renamed LG_ACC_INT
- net LG_ACC_INT: now also U7.11 (INT1)
- net EBUSY: no longer names the net of U1.14 (GPIO9)
- net ECS: no longer names the net of U1.11 (GPIO6)
- net EDC: no longer names the net of U1.12 (GPIO7)
- net ERESET: no longer names the net of U1.13 (GPIO8)
- net RTC_INT: no longer names the net of U1.19 (GPIO14)
- new net: U8.2 (NC), U8.3 (NC)
- no-connect marks 26 -> 32
Other:
- note added: "Buzzer"
- note added: "Check for address conflicts. Change SA0 if conflict"
- note added: "Gyroscope"
- note added: "High G Accelerometer"
- note added: "Low G Accelerometer"
- moved on the sheet: C2, C4, R1, SW1, SW2, U3

Commit message: i forgor
Parts:
- added AE1: NN02-101, besser_footprints:NN02-101_edge, symbol Device:Antenna
- added C20, C21: 2.7pF, Capacitor_SMD:C_0402_1005Metric, symbol Device:C
- added L1: 2.4nH, Capacitor_SMD:C_0402_1005Metric, symbol Device:L
Connections:
- net +3V3_2: now also C20.1, C21.2
- net RF_LNA_IN: now reaches U1.1 (LNA_IN)
- net RF_LNA_IN: now also C20.2, L1.1
- new net RF_ANT: AE1.1 (A), C21.1, L1.2
- no-connect marks 32 -> 31
Other:
- note added: "50Ω matching"
- note added: "Add power LED"
- note added: "Choose appropriate supercap"
- note added: "FDR Flash"
- note added: "See this issue about the WiFi transmit power being too high causing connectivity issues. This might be a hardware flaw, software fix in PyPaper repo. https://github.com/adafruit/circuitpython/pull/9369 https://discord.com/channels/327254708534116352/537365702651150357/1257897540314075177"
- moved on the sheet: C4, R1, SW2

Commit message: Change to IMU, start on buzzer, add magnetometer
Parts:
- removed AE1: NN02-101, besser_footprints:NN02-101_edge, symbol Device:Antenna
- removed L1: 2.4nH, Capacitor_SMD:C_0402_1005Metric, symbol Device:L
- removed SW2: PTS636 SK25F, Button_Switch_SMD:SW_Tactile_SPST_NO_Straight_CK_PTS636Sx25SMTRLFS, symbol Switch:SW_SPST
- removed U7: LIS3DH, Package_LGA:LGA-16_3x3mm_P0.5mm_LayoutBorder3x5y, symbol Sensor_Motion:LIS3DH
- added BZ1: Buzzer, symbol Device:Buzzer
- added Q2: DMP2045U-7, Package_TO_SOT_SMD:SOT-23-3, symbol Simulation_SPICE:PMOS
- added R10: 10k, Capacitor_SMD:C_0603_1608Metric, symbol Device:R
- added R8, R9: 100k, Capacitor_SMD:C_0603_1608Metric, symbol Device:R
- added TP1, TP2: TestPoint, symbol Connector:TestPoint
- added U7: LSM6DSO32, Package_LGA:LGA-14_3x2.5mm_P0.5mm_LayoutBorder3x4y, symbol Sensor_Motion:LSM6DSL
- added U9: LIS3MDL, Package_LGA:LGA-12_2x2mm_P0.5mm, symbol Sensor_Magnetic:LIS3MDL
- C10, C14, C15, C16, C7: value 10uf -> 10uF
- C20, C21: value 2.7pF -> 100nF; footprint Capacitor_SMD:C_0402_1005Metric -> Capacitor_SMD:C_0603_1608Metric
Connections:
- net +3V3_2: now also C20.2, BZ1.2 (-), R10.2, R9.1, TP2.1, U7.1 (SDO/SA0), U7.12 (CS), U7.2 (SDX), U7.3 (SCX), U7.5 (VDDIO), U7.6 (GND), U7.7 (GND), U7.8 (VDD), U9.10 (~{CS}), U9.12 (GND), U9.2 (GND), U9.3 (GND), U9.5 (Vdd), U9.6 (Vdd_IO), U9.9 (SDO/SA1)
- net RESET: now also TP1.1
- net SCL: now also U7.13 (SCL), U9.1 (SCL/SPC)
- net SDA: now also U7.14 (SDA), U9.11 (SDA/SDI/SDO)
- net VBAT: now also R8.2
- net VHIGH: now also Q2.2 (S)
- net BATT_INT renamed BAT_INT
- net LG_ACC_INT renamed IMU_INT
- net IMU_INT: now also U7.4 (INT1)
- net RF_ANT: no longer names the net of C21.1
- net RF_ANT: now also U9.4 (C1)
- net RF_LNA_IN: no longer names the net of U1.1 (LNA_IN)
- net RF_LNA_IN: no longer C20.2
- new net: BZ1.1 (+), Q2.3 (D)
- new net BUZZ: Q2.1 (G), R10.1
- new net VBAT_SENSE: R8.1, R9.2
Other:
- note added: "ADXL375 might be better"
- note added: "Ensure correct INT pin used"
- note added: "Low G Accel & Gyro"
- note added: "Magentometer"
- note added: "Not connected to MCU R values not set. Used to detect when running off of supercap to set error flag high."
- note added: "Not tested, this wiring may be incorrect (MOSFETs scary) Also get a better piezo zymbol"
- note added: "this is better than the slow battery monitor IC"
- note removed: "50Ω matching"
- note removed: "Add power LED"
- note removed: "Check for address conflicts. Change SA0 if conflict"
- note removed: "Gyroscope"
- note removed: "Low G Accelerometer"
- note removed: "See this issue about the WiFi transmit power being too high causing connectivity issues. This might be a hardware flaw, software fix in PyPaper repo. https://github.com/adafruit/circuitpython/pull/9369 https://discord.com/channels/327254708534116352/537365702651150357/1257897540314075177"
- moved on the sheet: C14, C17, C18, C19, C2, C7, C9, D2, J3, Q1, R7, U4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

Commit message: Add Flash and SD card SPI stuff
Parts:
- added C13: 100nF, Capacitor_SMD:C_0603_1608Metric, symbol Device:C
- added H1: M2.5_2.7mm, MountingHole:MountingHole_2.7mm_M2.5_Pad_Via, symbol Mechanical:MountingHole
- added J2: Micro_SD_Card_Det1, besser_footprints:GCT_MEM2061-01-188-00-A_REVA, symbol Connector:Micro_SD_Card_Det1
- added R11, R12, R13, R14, R15, R16: 47k, Capacitor_SMD:C_0603_1608Metric, symbol Device:R
- added U5: W25Q128JVPIQ, Package_SON:WSON-8-1EP_6x5mm_P1.27mm_EP3.4x4.3mm, symbol Memory_Flash:W25Q128JVS
- C15: renamed from C18; value 0.5 F -> 0.5F
- R6: renamed from R3; value 5.1k -> 10k
- R7: renamed from R4; value 5.1k -> 10k
- TP1: renamed from TP2; footprint (none) -> TestPoint:TestPoint_Pad_D1.5mm
- TP2: renamed from TP1; footprint (none) -> TestPoint:TestPoint_Pad_D1.5mm
- U6: renamed from U8; value H3LIS331DL -> H3LIS331DLTR; footprint (none) -> besser_footprints:TLGA-16L
- renumbered C12 to C10, C13 to C11, C17 to C12, C19 to C14, C7 to C16, C14 to C17, C15 to C18, C20 to C19, C4 to C2, C21 to C20, C16 to C21, C9 to C22, C5 to C4, C6 to C5, C8 to C6, C10 to C7, C2 to C8, C11 to C9, H3 to H2, H2 to H3, H1 to H4, J2 to J3, J3 to J4, Q2 to Q1, Q1 to Q2, R5 to R1, R9 to R10, R6 to R2, R1 to R3, R10 to R4, R2 to R5, R7 to R8, R8 to R9, U6 to U10, U3 to U2, U2 to U3, U7 to U4, U5 to U7, U9 to U8, U4 to U9
Connections:
- net +3V3_2: now also C13.1, C13.2, J2.10 (SHIELD), J2.4 (VDD), J2.6 (VSS), R11.1, R12.1, R13.1, R14.1, R15.1, R16.1, U5.4 (GND), U5.8 (VCC)
- net IMU_INT: now also U1.19 (GPIO14); no longer U1.6 (GPIO1)
- net IO11: no longer U1.16 (GPIO11)
- net IO12: no longer U1.17 (GPIO12)
- net IO13: no longer U1.18 (GPIO13)
- net MOSI: now also J2.3 (CMD), R13.2, U5.5 (DI(IO0))
- net SCK: now also U1.11 (GPIO6), J2.5 (CLK), R14.2, U5.6 (CLK); no longer U1.10 (GPIO5)
- net VHIGH: now also Q1.3 (D); no longer Q1.2 (S)
- net FSH_CS: now reaches U1.12 (GPIO7)
- net FSH_CS: now also U5.1 (~{CS})
- net SD_CS: now reaches U1.13 (GPIO8)
- net SD_CS: now also J2.2 (DAT3/CD), R12.2
- net at BZ1.1 (+): now also Q1.2 (S); no longer Q1.3 (D)
- net BAT_INT: no longer names the net of U1.27 (GPIO21)
- net BAT_INT: no longer U9.5 (~{ALRT})
- new net: J2.1 (DAT2), R11.2
- new net: J2.8 (DAT1), R16.2
- new net MISO: J2.7 (DAT0), R15.2, U1.10 (GPIO5), U5.2 (DO(IO1))
- no-connect marks 31 -> 35
Other:
- note added: "Can't use 35, 36, 37 on S3R8 as on-package PSRAM uses these for Octal SPI. In the future use external chip so we get back the GPIO pins from the SPI bus. (Also many Arduino libs dont let you use software SPI for some reason)"
- note added: "Flight Data Flash"
- note added: "Make better symbol."
- note added: "Must be initialized before other devices."
- note added: "Not tested, this wiring on pull up R may be incorrect (MOSFETs scary) Using a P channel FET, should maybe be N channel. Also get a better piezo zymbol"
- note added: "R values correct? ESP docs say 10k"
- note added: "SD Card"
- note added: "this is better than the slow battery monitor IC. Maybe get rid of it."
- note removed: "ADXL375 might be better"
- note removed: "Ensure correct INT pin used"
- note removed: "FDR Flash"
- note removed: "Not tested, this wiring may be incorrect (MOSFETs scary) Also get a better piezo zymbol"
- note removed: "this is better than the slow battery monitor IC"
- moved on the sheet: BZ1, C1, C11, C18, C20, C21, Q1, R4, R5, U10, U3

Commit message: do the shitfuck
Parts:
- removed C22: 100nF, Capacitor_SMD:C_0603_1608Metric, symbol Device:C
- removed J3: JST-SM04B-SRSS, besser_footprints:JST_SH_SM04B-SRSS-TB_1x04-1MP_P1.00mm_Horizontal, symbol Connector:Conn_01x04_Socket
- removed U9: MAX1704x, Package_DFN_QFN:TDFN-8-1EP_2x2mm_P0.5mm_EP0.8x1.2mm, symbol besserLib:MAX1704x
- added BZ2: Buzzer, symbol Device:Buzzer
- added D3: SS2040LL, Diode_SMD:D_SOD-123, symbol Diode:NSR0340HT1G
- added J5: JST-SM04B-SRSS, besser_footprints:JST_SH_SM04B-SRSS-TB_1x04-1MP_P1.00mm_Horizontal, symbol Connector:Conn_01x04_Socket
- added Q3: DMP2045U-7, Package_TO_SOT_SMD:SOT-23-3, symbol Simulation_SPICE:PMOS
- C15: value 0.5F -> 1.5F; footprint (none) -> besser_footprints:CP_Radial_D16.5mm_P12mm
Connections:
- net +3V3_2: now also J5.1 (Pin_1), Q3.2 (S)
- net BUZZ: now also Q3.1 (G)
- net SCL: now also J5.4 (Pin_4)
- net SDA: now also J5.3 (Pin_3)
- net VHIGH: now also BZ2.1 (+), D3.1 (K), J5.2 (Pin_2)
- new net: BZ2.2 (-), D3.2 (A), Q3.3 (D)
- no-connect marks 35 -> 34
Other:
- note added: "CARFIO Con."
- note added: "Not connected to Analog pin on MCU. R values not set. Used to detect when running off of supercap to set error flag high."
- note added: "Using 10k pullups, not 5.1k. Will this fix ocasional I2C setup error?"
- note removed: "Choose appropriate supercap"
- note removed: "GPIO"
- note removed: "Not connected to MCU R values not set. Used to detect when running off of supercap to set error flag high."
- note removed: "this is better than the slow battery monitor IC. Maybe get rid of it."
- moved on the sheet: BZ1, Q1, R10, R4, R9

Commit message: Finalize Schematic
Parts:
- removed BZ1: Buzzer, symbol Device:Buzzer
- removed H4: M2.5_2.7mm, MountingHole:MountingHole_2.7mm_M2.5_Pad_Via, symbol Mechanical:MountingHole
- removed Q1: DMP2045U-7, Package_TO_SOT_SMD:SOT-23-3, symbol Simulation_SPICE:PMOS
- removed R4: 10k, Capacitor_SMD:C_0603_1608Metric, symbol Device:R
- BZ1: renamed from BZ2; footprint (none) -> besser_footprints:CMT-9504-87-SMT_BUZZER
- R14: renamed from R9; value 100k -> 1k
- R15: renamed from R10; value 100k -> 806o
- renumbered C13 to C12, C12 to C13, C19 to C18, C18 to C19, D3 to D2, D2 to D3, J5 to J3, Q3 to Q1, R14 to R10, R15 to R11, R16 to R12, R8 to R13, R5 to R4, R6 to R5, R7 to R6, R11 to R7, R12 to R8, R13 to R9, U5 to U4, U4 to U5, U10 to U9
Connections:
- net VBAT_SENSE: now also U1.14 (GPIO9)
- net NEOPX renamed NEOPIXEL
Other:
- note added: "5v MAX"
- note added: "800/(1000+806e) = ~0.45 = 9/20 Power consumption: v^2/(R1+R2) = ~30mW"
- note added: "See: https://www.youtube.com/watch?v=FytOw9TRPcc"
- note removed: "Not connected to Analog pin on MCU. R values not set. Used to detect when running off of supercap to set error flag high."
- moved on the sheet: BZ1, D2, Q1, R6

Commit message: Tune schematic, start on PCB for eel on cod
Parts:
- added R4: 10K, Capacitor_SMD:C_0603_1608Metric, symbol Device:R
- added SW2: PTS636 SK25F, Button_Switch_SMD:SW_Tactile_SPST_NO_Straight_CK_PTS636Sx25SMTRLFS, symbol Switch:SW_SPST
- added TP3: TestPoint, TestPoint:TestPoint_Pad_D1.5mm, symbol Connector:TestPoint
- renumbered R9 to R10, R10 to R11, R11 to R12, R12 to R13, R13 to R14, R14 to R15, R15 to R16, R4 to R5, R5 to R6, R6 to R7, R7 to R8, R8 to R9
Connections:
- net +3V3_2: no longer C1.2, C10.2, C11.2, C12.2, C13.2, C14.2, C15.2, C16.1, C17.1, C18.2, C19.1, C2.2, C20.2, C21.2, C3.2, C4.2, C5.2, C6.2, C7.2, C8.1, C9.1, D1.2 (VSS), J1.A1 (GND), J1.A12 (GND), J1.B1 (GND), J1.B12 (GND), J2.10 (SHIELD), J2.6 (VSS), J3.1 (Pin_1), J4.2 (Pin_2), Q1.2 (S), R1.2, R14.2, R16.1, R2.2, SW1.2 (B), TP1.1, U1.57 (GND), U2.3 (VSS), U2.8 (VSS), U2.9 (VSS), U3.4 (GND), U4.4 (GND), U5.1 (SDO/SA0), U5.2 (SDX), U5.3 (SCX), U5.6 (GND), U5.7 (GND), U6.10 (NC), U6.12 (GND), U6.13 (GND), U6.16 (GND), U6.5 (GND), U6.7 (SA0), U7.2 (GND), U8.12 (GND), U8.2 (GND), U8.3 (GND), U8.9 (SDO/SA1), U9.2 (GND), Y1.2, Y1.4
- net BUZZ: now also R4.2
- net IO11: now also TP1.1, U1.16 (GPIO11)
- net IO12: now also TP2.1, U1.17 (GPIO12)
- net IO13: now also U1.18 (GPIO13), TP3.1
- net RESET: now also SW2.2 (B); no longer TP2.1
- net GND: now reaches U6.10 (NC)
- net GND: now also C1.2, C10.2, C11.2, C12.2, C13.2, C14.2, C15.2, C16.1, C17.1, C18.2, C19.1, C2.2, C20.2, C21.2, C3.2, C4.2, C5.2, C6.2, C7.2, C8.1, C9.1, D1.2 (VSS), J1.A1 (GND), J1.A12 (GND), J1.B1 (GND), J1.B12 (GND), J2.10 (SHIELD), J2.6 (VSS), J3.1 (Pin_1), J4.2 (Pin_2), Q1.2 (S), R1.2, R14.2, R16.1, R2.2, SW1.2 (B), U1.57 (GND), U2.3 (VSS), U2.8 (VSS), U2.9 (VSS), U3.4 (GND), U4.4 (GND), U5.1 (SDO/SA0), U5.2 (SDX), U5.3 (SCX), U5.6 (GND), U5.7 (GND), U6.12 (GND), U6.13 (GND), U6.16 (GND), U6.5 (GND), U6.7 (SA0), U7.2 (GND), U8.12 (GND), U8.2 (GND), U8.3 (GND), U8.9 (SDO/SA1), U9.2 (GND), Y1.2, Y1.4, R4.1, SW2.1 (A)
- no-connect marks 34 -> 37
Other:
- note added: "800/(1000+806) = ~0.45 = 9/20 Power consumption: v^2/(R1+R2) = ~30mW"
- note added: "GPIO"
- note added: "Not tested, this pull down R may be required as this is a P channel FET."
- note removed: "800/(1000+806e) = ~0.45 = 9/20 Power consumption: v^2/(R1+R2) = ~30mW"
- note removed: "Not tested, this wiring on pull up R may be incorrect (MOSFETs scary) Using a P channel FET, should maybe be N channel. Also get a better piezo zymbol"
- company: Chugnus Aerospace -> Chungus Aerospace
- moved on the sheet: J3

Commit message: Redo power
Parts:
- removed C19, C21, C7: 10uF, Capacitor_SMD:C_0603_1608Metric, symbol Device:C
- removed H3: M2.5_2.7mm, MountingHole:MountingHole_2.7mm_M2.5_Pad_Via, symbol Mechanical:MountingHole
- removed TP3: TestPoint, TestPoint:TestPoint_Pad_D1.5mm, symbol Connector:TestPoint
- removed U7, U9: AP2112K-3.3TRG1, Package_TO_SOT_SMD:SOT-23-5, symbol Regulator_Linear:AP2112K-3.3
- added U7: NCP187AMT330TAG, besser_footprints:6-WDFN_2x2mm_EP, symbol besserLib:NCP187
- C15: renamed from C16; value 10uF -> 1uF
- H1, H2: footprint MountingHole:MountingHole_2.7mm_M2.5_Pad_Via -> besser_footprints:M2.5_2.7mm_hole
- renumbered C11 to C10, C12 to C11, C13 to C12, C14 to C13, C15 to C14, C17 to C16, C18 to C17, C20 to C18, C8 to C7, C9 to C8, C10 to C9
Connections:
- net +3V3_MCU is gone; now on net +3V3: C16.2, C3.1, C4.1, C5.1, C6.1, R3.2, U1.2 (VDD3P3), U1.20 (VDD3P3_RTC), U1.3 (VDD3P3), U1.46 (VDD3P3_CPU), U1.55 (VDDA), U1.56 (VDDA)
- net FSH_CS: now also U1.14 (GPIO9); no longer U1.12 (GPIO7)
- net GND: now also U7.3 (GND), U7.EP
- net IO11: now also TP2.1; no longer TP1.1
- net IO12: no longer TP2.1, U1.17 (GPIO12)
- net IO13: no longer U1.18 (GPIO13)
- net MISO: now also U1.11 (GPIO6); no longer U1.10 (GPIO5)
- net MOSI: now also U1.10 (GPIO5); no longer U1.9 (GPIO4)
- net NEOPIXEL: now also U1.6 (GPIO1); no longer U1.15 (GPIO10)
- net SCK: now also U1.12 (GPIO7); no longer U1.11 (GPIO6)
- net VBAT_SENSE: now also U1.9 (GPIO4); no longer U1.14 (GPIO9)
- net VHIGH: now also U7.1 (VIN), U7.2 (EN)
- net +3V3_2 renamed +3V3
- net +3V3: now also U7.5 (SNS), U7.6 (VOUT)
- net IMU_INT: no longer names the net of U1.19 (GPIO14)
- net IMU_INT: no longer U5.4 (INT1)
- new net IO10: TP1.1, U1.15 (GPIO10)
- no-connect marks 37 -> 41
Other:
- moved on the sheet: C14, C15, C16, D3, J4, Q2, R14, R15, R16
