File: AC-FR/ACFR-PCB/ACFR-PCB.kicad_sch (KiCad schematic)
At the start: 59 parts, among them J1 USB4105-GF-A, J2 Micro_SD_Card_Det1, J4 JST-PH, Q1 DMP2045U-7, Q2 DMP2045U-7, SW1 PTS636 SK25F, SW2 PTS636 SK25F, U1 ESP32-S3R8, U2 BMP390, U3 W25Q128JVPIQ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

Commit message: Work on routing
Connections:
- net IO11: now also U1.15 (GPIO10); no longer U1.16 (GPIO11)
- net IO4: now reaches U1.9 (GPIO4)
- net IO4: now also TP1.1
- removed net IO10: TP1.1, U1.15 (GPIO10)

Commit message: Continue work on routing
Parts:
- added J3: JST-SM04B-SRSS, besser_footprints:JST_SH_SM04B-SRSS-TB_1x04-1MP_P1.00mm_Horizontal, symbol Connector:Conn_01x04_Socket
Connections:
- net GND: now also J3.1 (Pin_1)
- net SCL: now also J3.4 (Pin_4)
- net SDA: now also J3.3 (Pin_3)
- net VHIGH: now also J3.2 (Pin_2)
Other:
- note added: "CARFIO Con."
- note added: "For the CARFIO Radio. NOT any other GPIO device, as it uses VHIGH."
Changed lines of the file:
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@@
 	(wire
 		(pts
+			(xy 237.49 265.43) (xy 233.68 265.43)
+		)
+		(stroke
+			(width 0)
+			(type default)
+		)
+	)
+	(wire
+		(pts
 			(xy 132.08 38.1) (xy 132.08 35.56)
 		)
@@
 	(wire
 		(pts
+			(xy 227.33 270.51) (xy 237.49 270.51)
+		)
+		(stroke
+			(width 0)
+			(type default)
+		)
+	)
+	(wire
+		(pts
 			(xy 158.75 251.46) (xy 167.64 251.46)
 		)
@@
 	(polyline
 		(pts
+			(xy 224.79 284.48) (xy 224.79 252.73)
+		)
+		(stroke
+			(width 0)
+			(type dash)
+		)
+	)
+	(polyline
+		(pts
 			(xy 13.97 76.2) (xy 86.36 76.2)
 		)
@@
 		)
 	)
+	(polyline
+		(pts
+			(xy 224.79 252.73) (xy 274.32 252.73)
+		)
+		(stroke
+			(width 0)
+			(type dash)
+		)
+	)
 	(wire
 		(pts
@@
 	(wire
 		(pts
+			(xy 233.68 267.97) (xy 237.49 267.97)
+		)
+		(stroke
+			(width 0)
+			(type default)
+		)
+	)
+	(wire
+		(pts
 			(xy 77.47 166.37) (xy 90.17 166.37)
 		)
@@
 	(text "5v MAX"
 		(exclude_from_sim no)
-		(at 362.204 206.248 0)
+		(at 363.982 204.47 0)
 		(effects
 			(font
@@
 		)
 	)
+	(text "CARFIO Con.\n"
+		(exclude_from_sim no)
+		(at 249.428 259.08 0)
+		(effects
+			(font
+				(size 5.08 5.08)
+			)
+		)
+	)
 	(text "USB-C\n"
 		(exclude_from_sim no)
@@
 		)
 	)
+	(text "For the CARFIO\nRadio. NOT\nany other GPIO\ndevice, as it \nuses VHIGH.\n"
+		(exclude_from_sim no)
+		(at 260.35 269.748 0)
+		(effects
+			(font
+				(size 1.27 1.27)
+			)
+		)
+	)
 	(text "See:\nhttps://www.youtube.com/watch?v=FytOw9TRPcc"
 		(exclude_from_sim no)
@@
 		)
 	)
+	(label "VHIGH"
+		(at 227.33 270.51 0)
+		(fields_autoplaced yes)
+		(effects
+			(font
+				(size 1.27 1.27)
+			)
+			(justify left bottom)
+		)
+	)
 	(label "SDA"
 		(at 254 45.72 0)
@@
 	)
 	(label "SCL"
+		(at 233.68 265.43 0)
+		(fields_autoplaced yes)
+		(effects
+			(font
+				(size 1.27 1.27)
+			)
+			(justify left bottom)
+		)
+	)
+	(label "SCL"
 		(at 341.63 44.45 0)
 		(fields_autoplaced yes)
@@
 		)
 	)
+	(label "SDA"
+		(at 233.68 267.97 0)
+		(fields_autoplaced yes)
+		(effects
+			(font
+				(size 1.27 1.27)
+			)
+			(justify left bottom)
+		)
+	)
 	(label "SPICS0"
 		(at 129.54 198.12 0)
@@
 	)
 	(symbol
+		(lib_id "Connector:Conn_01x04_Socket")
+		(at 242.57 270.51 0)
+		(mirror x)
+		(unit 1)
+		(exclude_from_sim no)
+		(in_bom yes)
+		(on_board yes)
+		(dnp no)
+		(property "Reference" "J3"
+			(at 244.094 270.764 0)
+			(effects
+				(font
+					(size 1.27 1.27)
+				)
+				(justify left)
+			)
+		)
+		(property "Value" "JST-SM04B-SRSS"
+			(at 230.378 276.86 0)
+			(effects
+				(font
+					(size 1.27 1.27)
+				)
+				(justify left)
+			)
+		)
+		(property "Footprint" "besser_footprints:JST_SH_SM04B-SRSS-TB_1x04-1MP_P1.00mm_Horizontal"
+			(at 242.57 270.51 0)
+			(effects
+				(font
+					(size 1.27 1.27)
+				)
+				(hide yes)
+			)
+		)
+		(property "Datasheet" "~"
+			(at 242.57 270.51 0)
+			(effects
+				(font
+					(size 1.27 1.27)
+				)
+				(hide yes)
+			)
+		)
+		(property "Description" "Generic connector, single row, 01x04, script generated"
+			(at 242.57 270.51 0)
+			(effects
+				(font
+					(size 1.27 1.27)
+				)
+				(hide yes)
+			)
+		)
+		(pin "1"
+		)
+		(pin "2"
+		)
+		(pin "3"
+		)
+		(pin "4"
+		)
+		(instances
+			(project "ACFR-PCB"
+				(path "/8287cc23-38e5-458d-8ed1-870f124a9a59"
+					(reference "J3")
+					(unit 1)
+				)
+			)
+		)
+	)
+	(symbol
 		(lib_id "power:+5V")
 		(at 351.79 209.55 0)
@@
 					(unit 1)
 				)
+			)
+		)
+	)
+	(symbol
+		(lib_id "power:GND")
+		(at 237.49 273.05 0)
+		(unit 1)
+		(exclude_from_sim no)
+		(in_bom yes)
+		(on_board yes)
+		(dnp no)
+		(fields_autoplaced yes)
+		(property "Reference" "#PWR046"
+			(at 237.49 279.4 0)
+			(effects
+				(font
+					(size 1.27 1.27)
+				)
+				(hide yes)
+			)
+		)
+		(property "Value" "GND"
+			(at 237.49 278.13 0)
+			(effects
+				(font
+					(size 1.27 1.27)
+				)
+				(hide yes)
+			)
+		)
+		(property "Footprint" ""
+			(at 237.49 273.05 0)
+			(effects
+				(font
+					(size 1.27 1.27)
+				)
+				(hide yes)
+			)
+		)
+		(property "Datasheet" ""
+			(at 237.49 273.05 0)
+			(effects
+				(font
+					(size 1.27 1.27)
+				)
+				(hide yes)
+			)
+		)
+		(property "Description" "Power symbol creates a global label with name \"GND\" , ground"
+			(at 237.49 273.05 0)
+			(effects
+				(font
+					(size 1.27 1.27)
+				)
+				(hide yes)
+			)
+		)
+		(pin "1"
+		)
+		(instances
+			(project "ACFR-PCB"
+				(path "/8287cc23-38e5-458d-8ed1-870f124a9a59"
+					(reference "#PWR046")
+					(unit 1)
+				)

Commit message: ACFR R1
Parts:
- removed Q1: DMP2045U-7, Package_TO_SOT_SMD:SOT-23-3, symbol Simulation_SPICE:PMOS
- added Q1: NXV55UNR, Package_TO_SOT_SMD:SOT-23-3, symbol Simulation_SPICE:NMOS
- R4: now fitted
- R8: value 47k -> 100k
Connections:
- net BUZZ: now also Q1.1 (G)
- net GND: now also Q1.2 (S)
- net at BZ1.2 (-), D2.2 (A): now also Q1.3 (D)
Other:
- note removed: "Make better symbol."
- note removed: "Not tested, this pull down R may be required as this is a P channel FET."
- note removed: "TODO: Investigate flash usage to make sure everything will work with Adafruit flash lib and Arduino SD lib"
Changed lines of the file:
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@@
 	(title_block
 		(title "Aerochungus Flight Recorder")
-		(date "2024-10-29")
+		(date "2024-11-06")
 		(rev "R1")
 		(company "Chungus Aerospace")
@@
 		)
 	)
-	(text "TODO:\nInvestigate flash usage to make \nsure everything will work with \nAdafruit flash lib\nand Arduino SD lib\n"
-		(exclude_from_sim no)
-		(at 234.95 158.75 0)
-		(effects
-			(font
-				(size 5.08 5.08)
-			)
-		)
-	)
 	(text "Switches\n"
 		(exclude_from_sim no)
@@
 		)
 	)
-	(text "Not tested, this\npull down R may be\nrequired as this is\na P channel FET."
-		(exclude_from_sim no)
-		(at 141.224 120.904 0)
-		(effects
-			(font
-				(size 1.27 1.27)
-			)
-		)
-	)
 	(text "MCU"
 		(exclude_from_sim no)
@@
 		)
 	)
-	(text "Make better symbol."
-		(exclude_from_sim no)
-		(at 229.362 124.714 0)
-		(effects
-			(font
-				(size 1.905 1.905)
-			)
-		)
-	)
 	(text "Must be initialized\nbefore other devices."
 		(exclude_from_sim no)
@@
 		)
 	)
-	(label "IO14"
-		(at 24.13 222.25 0)
-		(fields_autoplaced yes)
-		(effects
-			(font
-				(size 1.27 1.27)
-			)
-			(justify left bottom)
-		)
-	)
 	(label "SCK"
 		(at 160.02 100.33 0)
@@
 		)
 	)
-	(label "IO1"
-		(at 24.13 189.23 0)
-		(fields_autoplaced yes)
-		(effects
-			(font
-				(size 1.27 1.27)
-			)
-			(justify left bottom)
-		)
-	)
 	(label "SD_CS"
 		(at 241.3 100.33 0)
@@
 		)
 	)
-	(label "IO12"
-		(at 24.13 217.17 0)
-		(fields_autoplaced yes)
-		(effects
-			(font
-				(size 1.27 1.27)
-			)
-			(justify left bottom)
-		)
-	)
-	(label "IO21"
-		(at 24.13 234.95 0)
-		(fields_autoplaced yes)
-		(effects
-			(font
-				(size 1.27 1.27)
-			)
-			(justify left bottom)
-		)
-	)
 	(label "NEOPIXEL"
 		(at 21.59 142.24 0)
@@
 	)
 	(symbol
+		(lib_id "Simulation_SPICE:NMOS")
+		(at 115.57 110.49 0)
+		(unit 1)
+		(exclude_from_sim no)
+		(in_bom yes)
+		(on_board yes)
+		(dnp no)
+		(property "Reference" "Q1"
+			(at 120.904 111.76 0)
+			(effects
+				(font
+					(size 1.27 1.27)
+				)
+				(justify left)
+			)
+		)
+		(property "Value" "NXV55UNR"
+			(at 120.904 109.474 0)
+			(effects
+				(font
+					(size 1.27 1.27)
+				)
+				(justify left)
+			)
+		)
+		(property "Footprint" "Package_TO_SOT_SMD:SOT-23-3"
+			(at 120.65 107.95 0)
+			(effects
+				(font
+					(size 1.27 1.27)
+				)
+				(hide yes)
+			)
+		)
+		(property "Datasheet" "https://www.digikey.com/en/products/detail/nexperia-usa-inc/NXV55UNR/13898532"
+			(at 115.57 123.19 0)
+			(effects
+				(font
+					(size 1.27 1.27)
+				)
+				(hide yes)
+			)
+		)
+		(property "Description" "N-MOSFET transistor, drain/source/gate"
+			(at 115.57 110.49 0)
+			(effects
+				(font
+					(size 1.27 1.27)
+				)
+				(hide yes)
+			)
+		)
+		(property "Sim.Device" "NMOS"
+			(at 115.57 127.635 0)
+			(effects
+				(font
+					(size 1.27 1.27)
+				)
+				(hide yes)
+			)
+		)
+		(property "Sim.Type" "VDMOS"
+			(at 115.57 129.54 0)
+			(effects
+				(font
+					(size 1.27 1.27)
+				)
+				(hide yes)
+			)
+		)
+		(property "Sim.Pins" "1=G 2=S 3=D"
+			(at 115.57 125.73 0)
+			(effects
+				(font
+					(size 1.27 1.27)
+				)
+				(hide yes)
+			)
+		)
+		(pin "3"
+		)
+		(pin "1"
+		)
+		(pin "2"
+		)
+		(instances
+			(project "ACFR-PCB"
+				(path "/8287cc23-38e5-458d-8ed1-870f124a9a59"
+					(reference "Q1")
+					(unit 1)
+				)
+			)
+		)
+	)
+	(symbol
 		(lib_id "power:GND")
 		(at 62.23 113.03 0)
@@
 	)
 	(symbol
-		(lib_id "Simulation_SPICE:PMOS")
-		(at 115.57 110.49 0)
-		(unit 1)
-		(exclude_from_sim no)
-		(in_bom yes)
-		(on_board yes)
-		(dnp no)
-		(fields_autoplaced yes)
-		(property "Reference" "Q1"
-			(at 121.92 109.22 0)
-			(effects
-				(font
-					(size 1.27 1.27)
-				)
-				(justify left)
-			)
-		)
-		(property "Value" "DMP2045U-7"
-			(at 121.92 111.76 0)
-			(effects
-				(font
-					(size 1.27 1.27)
-				)
-				(justify left)
-			)
-		)
-		(property "Footprint" "Package_TO_SOT_SMD:SOT-23-3"
-			(at 120.65 107.95 0)
-			(effects
-				(font
-					(size 1.27 1.27)
-				)
-				(hide yes)
-			)
-		)
-		(property "Datasheet" "https://www.digikey.com/en/products/detail/diodes-incorporated/DMP2045U-7/8275356"
-			(at 115.57 123.19 0)
-			(effects
-				(font
-					(size 1.27 1.27)
-				)
-				(hide yes)
-			)
-		)
-		(property "Description" "P-MOSFET transistor, drain/source/gate"
-			(at 115.57 110.49 0)
-			(effects
-				(font
-					(size 1.27 1.27)
-				)
-				(hide yes)
-			)
-		)
-		(property "Sim.Device" "PMOS"
-			(at 115.57 127.635 0)
-			(effects
-				(font
-					(size 1.27 1.27)
-				)
-				(hide yes)
-			)
-		)
-		(property "Sim.Type" "VDMOS"
-			(at 115.57 129.54 0)
-			(effects
-				(font
-					(size 1.27 1.27)
-				)
-				(hide yes)
-			)
-		)
-		(property "Sim.Pins" "1=G 2=S 3=D"
-			(at 115.57 125.73 0)
-			(effects
-				(font
-					(size 1.27 1.27)
-				)
-				(hide yes)
-			)
-		)
-		(pin "2"
-		)
-		(pin "3"
-		)
-		(pin "1"
-		)
-		(instances
-			(project "ACFR-PCB"
-				(path "/8287cc23-38e5-458d-8ed1-870f124a9a59"
-					(reference "Q1")
-					(unit 1)
-				)
-			)
-		)
-	)
-	(symbol
 		(lib_id "power:GND")
 		(at 360.68 59.69 0)
@@
 		(in_bom yes)
 		(on_board yes)
-		(dnp yes)
+		(dnp no)
 		(property "Reference" "R4"
 			(at 110.744 114.3 0)
@@
 		)
 		(property "Value" "10K"
-			(at 108.204 114.3 90)
+			(at 107.95 114.3 90)
 			(effects
 				(font
@@
 			)
 		)
-		(property "Datasheet" "~"
+		(property "Datasheet" "https://www.digikey.com/en/products/detail/c-k/PTS636-SK25F-SMTR-LFS/10071743"
 			(at 53.34 105.41 0)
 			(effects
@@
 			)
 		)
-		(property "Value" "47k"
-			(at 168.91 91.186 90)
+		(property "Value" "100k"
+			(at 168.91 90.678 90)
 			(effects
 				(font
@@
 			)
 		)
-		(property "Datasheet" "~"
+		(property "Datasheet" "https://www.digikey.com/en/products/detail/c-k/PTS636-SK25F-SMTR-LFS/10071743"
 			(at 21.59 105.41 0)
 			(effects

Commit message: stuff
Parts:
- added TP3, TP4, TP5: TestPoint, TestPoint:TestPoint_Pad_1.0x1.0mm, symbol Connector:TestPoint
Connections:
- net +3V3: now also TP3.1
- net SCL: now also TP4.1
- net SDA: now also TP5.1
Other:
- note removed: "Using 10k pullups, not 5.1k. Will this fix ocasional I2C setup error?"
Changed lines of the file:
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@@
 	(title_block
 		(title "Aerochungus Flight Recorder")
-		(date "2024-11-06")
-		(rev "R1")
+		(date "2024-11-16")
+		(rev "R2")
 		(company "Chungus Aerospace")
 	)
@@
 	)
 	(junction
+		(at 151.13 170.18)
+		(diameter 0)
+		(color 0 0 0 0)
+	)
+	(junction
 		(at 106.68 45.72)
 		(diameter 0)
@@
 	)
 	(junction
+		(at 151.13 162.56)
+		(diameter 0)
+		(color 0 0 0 0)
+	)
+	(junction
 		(at 360.68 33.02)
 		(diameter 0)
@@
 	(wire
 		(pts
-			(xy 148.59 170.18) (xy 153.67 170.18)
+			(xy 144.78 170.18) (xy 151.13 170.18)
 		)
 		(stroke
@@
 	(wire
 		(pts
+			(xy 151.13 170.18) (xy 153.67 170.18)
+		)
+		(stroke
+			(width 0)
+			(type default)
+		)
+	)
+	(wire
+		(pts
 			(xy 351.79 231.14) (xy 367.03 231.14)
 		)
@@
 		)
 	)
+	(wire
+		(pts
+			(xy 151.13 162.56) (xy 153.67 162.56)
+		)
+		(stroke
+			(width 0)
+			(type default)
+		)
+	)
 	(polyline
 		(pts
@@
 	(wire
 		(pts
-			(xy 148.59 162.56) (xy 153.67 162.56)
+			(xy 144.78 162.56) (xy 151.13 162.56)
 		)
 		(stroke
@@
 		)
 	)
-	(text "Using 10k pullups,\nnot 5.1k.\n\nWill this fix\nocasional I2C\nsetup error?"
-		(exclude_from_sim no)
-		(at 156.21 150.114 0)
-		(effects
-			(font
-				(size 1.27 1.27)
-			)
-		)
-	)
 	(text "Magentometer"
 		(exclude_from_sim no)
@@
 	)
 	(label "SCL"
-		(at 148.59 170.18 0)
+		(at 144.78 170.18 0)
 		(fields_autoplaced yes)
 		(effects
@@
 	)
 	(label "SDA"
-		(at 148.59 162.56 0)
+		(at 144.78 162.56 0)
 		(fields_autoplaced yes)
 		(effects
@@
 	)
 	(symbol
+		(lib_id "Connector:TestPoint")
+		(at 151.13 162.56 0)
+		(unit 1)
+		(exclude_from_sim no)
+		(in_bom yes)
+		(on_board yes)
+		(dnp no)
+		(property "Reference" "TP5"
+			(at 149.352 156.972 0)
+			(effects
+				(font
+					(size 1.27 1.27)
+				)
+				(justify left)
+			)
+		)
+		(property "Value" "TestPoint"
+			(at 146.05 162.306 90)
+			(effects
+				(font
+					(size 1.27 1.27)
+				)
+				(justify left)
+				(hide yes)
+			)
+		)
+		(property "Footprint" "TestPoint:TestPoint_Pad_1.0x1.0mm"
+			(at 156.21 162.56 0)
+			(effects
+				(font
+					(size 1.27 1.27)
+				)
+				(hide yes)
+			)
+		)
+		(property "Datasheet" "~"
+			(at 156.21 162.56 0)
+			(effects
+				(font
+					(size 1.27 1.27)
+				)
+				(hide yes)
+			)
+		)
+		(property "Description" "test point"
+			(at 151.13 162.56 0)
+			(effects
+				(font
+					(size 1.27 1.27)
+				)
+				(hide yes)
+			)
+		)
+		(pin "1"
+		)
+		(instances
+			(project "ACFR-PCB"
+				(path "/8287cc23-38e5-458d-8ed1-870f124a9a59"
+					(reference "TP5")
+					(unit 1)
+				)
+			)
+		)
+	)
+	(symbol
 		(lib_id "power:GND")
 		(at 373.38 33.02 0)
@@
 	)
 	(symbol
+		(lib_id "Connector:TestPoint")
+		(at 151.13 170.18 180)
+		(unit 1)
+		(exclude_from_sim no)
+		(in_bom yes)
+		(on_board yes)
+		(dnp no)
+		(property "Reference" "TP4"
+			(at 152.654 175.768 0)
+			(effects
+				(font
+					(size 1.27 1.27)
+				)
+				(justify left)
+			)
+		)
+		(property "Value" "TestPoint"
+			(at 156.21 170.434 90)
+			(effects
+				(font
+					(size 1.27 1.27)
+				)
+				(justify left)
+				(hide yes)
+			)
+		)
+		(property "Footprint" "TestPoint:TestPoint_Pad_1.0x1.0mm"
+			(at 146.05 170.18 0)
+			(effects
+				(font
+					(size 1.27 1.27)
+				)
+				(hide yes)
+			)
+		)
+		(property "Datasheet" "~"
+			(at 146.05 170.18 0)
+			(effects
+				(font
+					(size 1.27 1.27)
+				)
+				(hide yes)
+			)
+		)
+		(property "Description" "test point"
+			(at 151.13 170.18 0)
+			(effects
+				(font
+					(size 1.27 1.27)
+				)
+				(hide yes)
+			)
+		)
+		(pin "1"
+		)
+		(instances
+			(project "ACFR-PCB"
+				(path "/8287cc23-38e5-458d-8ed1-870f124a9a59"
+					(reference "TP4")
+					(unit 1)
+				)
+			)
+		)
+	)
+	(symbol
 		(lib_id "Connector:Conn_01x04_Socket")
 		(at 242.57 270.51 0)
@@
 					(unit 1)
 				)
+			)
+		)
+	)
+	(symbol
+		(lib_id "Connector:TestPoint")
+		(at 396.24 231.14 0)
+		(unit 1)
+		(exclude_from_sim no)
+		(in_bom yes)
+		(on_board yes)
+		(dnp no)
+		(property "Reference" "TP3"
+			(at 396.24 226.314 90)
+			(effects
+				(font
+					(size 1.27 1.27)
+				)
+				(justify left)
+			)
+		)
+		(property "Value" "TestPoint"
+			(at 391.16 230.886 90)
+			(effects
+				(font
+					(size 1.27 1.27)
+				)
+				(justify left)
+				(hide yes)
+			)
+		)
+		(property "Footprint" "TestPoint:TestPoint_Pad_1.0x1.0mm"
+			(at 401.32 231.14 0)
+			(effects
+				(font
+					(size 1.27 1.27)
+				)
+				(hide yes)
+			)
+		)
+		(property "Datasheet" "~"
+			(at 401.32 231.14 0)
+			(effects
+				(font
+					(size 1.27 1.27)
+				)
+				(hide yes)
+			)
+		)
+		(property "Description" "test point"
+			(at 396.24 231.14 0)
+			(effects
+				(font
+					(size 1.27 1.27)
+				)
+				(hide yes)
+			)
+		)
+		(pin "1"
+		)
+		(instances
+			(project "ACFR-PCB"
+				(path "/8287cc23-38e5-458d-8ed1-870f124a9a59"
+					(reference "TP3")
+					(unit 1)
+				)
