File: AC-FR/ACFR-PCB/_autosave-ACFR-PCB.kicad_sch (KiCad schematic)
At the start: 56 parts, among them J1 USB4105-GF-A, J2 Micro_SD_Card_Det1, J4 JST-PH, Q1 DMP2045U-7, Q2 DMP2045U-7, SW1 PTS636 SK25F, U1 ESP32-S3R8, U2 BMP390, U3 W25Q128JVPIQ, U4 W25Q128JVPIQ, U5 LSM6DSO32, U6 H3LIS331DLTR, U7 LIS3MDL, U8 NCP187AMT330TAG, Y1 ECS-400-8-36B-7KY

Commit message: Work on routing
Parts:
- added C2: 1uF, Capacitor_SMD:C_0603_1608Metric, symbol Device:C
- added R3: 5.1K, Capacitor_SMD:C_0603_1608Metric, symbol Device:R
- added SW2: PTS636 SK25F, Button_Switch_SMD:SW_Tactile_SPST_NO_Straight_CK_PTS636Sx25SMTRLFS, symbol Switch:SW_SPST
- TP1, TP2: footprint TestPoint:TestPoint_Pad_D1.5mm -> TestPoint:TestPoint_Pad_1.0x1.0mm
Connections:
- net +3V3: now also R3.2; no longer U1.4 (CHIP_PU)
- net BUZZ: now also U1.51 (GPIO45)
- net FSH_CS: now also U1.12 (GPIO7); no longer U1.14 (GPIO9)
- net GND: now also C2.2, SW2.1 (A)
- net IO11: now also U1.15 (GPIO10); no longer U1.16 (GPIO11)
- net MISO: now also U1.11 (GPIO6); no longer U1.13 (GPIO8)
- net MOSI: now also U1.13 (GPIO8); no longer U1.11 (GPIO6)
- net SCK: now also U1.14 (GPIO9); no longer U1.12 (GPIO7)
- net IO4: now reaches U1.9 (GPIO4)
- net IO4: now also TP1.1
- removed net IO10: TP1.1, U1.15 (GPIO10)
- new net RESET: C2.1, R3.1, SW2.2 (B), U1.4 (CHIP_PU)
Other:
- note added: "Switches"
- moved on the sheet: SW1

Commit message: Continue work on routing
Parts:
- added J3: JST-SM04B-SRSS, besser_footprints:JST_SH_SM04B-SRSS-TB_1x04-1MP_P1.00mm_Horizontal, symbol Connector:Conn_01x04_Socket
- added U9: ZOE-M8Q, RF_GPS:ublox_ZOE_M8, symbol RF_GPS:ZOE-M8Q
Connections:
- net GND: now also J3.1 (Pin_1)
- net SCL: now also J3.4 (Pin_4)
- net SDA: now also J3.3 (Pin_3)
- net VHIGH: now also J3.2 (Pin_2)
- new net: U9.A1 (GND), U9.A3 (GND), U9.A5 (GND), U9.A7 (GND), U9.A8 (GND), U9.A9 (GND), U9.B9 (GND), U9.C7 (GND), U9.C9 (GND), U9.D6 (GND), U9.D9 (GND), U9.E7 (GND), U9.F7 (GND), U9.G3 (GND), U9.G6 (GND), U9.G7 (GND), U9.J3 (GND), U9.J9 (GND)
- new net: U9.J1 (VCC), U9.J2 (VCC)
Other:
- note added: "CARFIO Con."
- note added: "For the CARFIO Radio. NOT any other GPIO device, as it uses VHIGH."
