File: AC-FR/backup/ACFR-PCB.kicad_sch (KiCad schematic)
At the start: 59 parts, among them J1 USB4105-GF-A, J2 Micro_SD_Card_Det1, J4 JST-PH, Q1 DMP2045U-7, Q2 DMP2045U-7, SW1 PTS636 SK25F, SW2 PTS636 SK25F, U1 ESP32-S3R8, U2 BMP390, U3 W25Q128JVPIQ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

Commit message: Finally make progress on layout and routing
Parts:
- removed C2: 1uF, Capacitor_SMD:C_0603_1608Metric, symbol Device:C
- removed R3: 5.1K, Capacitor_SMD:C_0603_1608Metric, symbol Device:R
- removed SW2: PTS636 SK25F, Button_Switch_SMD:SW_Tactile_SPST_NO_Straight_CK_PTS636Sx25SMTRLFS, symbol Switch:SW_SPST
- TP1, TP2: footprint TestPoint:TestPoint_Pad_1.0x1.0mm -> TestPoint:TestPoint_Pad_D1.5mm
Connections:
- net RESET is gone; now on net +3V3: U1.4 (CHIP_PU)
- net BUZZ: no longer U1.51 (GPIO45)
- net FSH_CS: now also U1.14 (GPIO9); no longer U1.12 (GPIO7)
- net MISO: now also U1.13 (GPIO8); no longer U1.11 (GPIO6)
- net MOSI: now also U1.11 (GPIO6); no longer U1.13 (GPIO8)
- net SCK: now also U1.12 (GPIO7); no longer U1.14 (GPIO9)
Other:
- note removed: "Switches"
- moved on the sheet: SW1
